Commit message: working on gps integration

File: SC-LIO-SAM/launch/include/config/robot.urdf.xacro (robot description, xacro)
@@ -9,8 +9,8 @@
     <origin xyz="0 0 0" rpy="0 0 0" />
   </joint>
-  <link name="imu_link"> </link>
+  <link name="sensor"> </link>
   <joint name="imu_joint" type="fixed">
     <parent link="chassis_link" />
-    <child link="imu_link" />
+    <child link="sensor" />
     <origin xyz="0 0 0" rpy="0 0 0" />
   </joint>
@@ -21,8 +21,8 @@
     <origin xyz="0 0 0" rpy="0 0 0" />
   </joint>
-  <link name="navsat_link"> </link>
+  <link name="gps"> </link>
   <joint name="navsat_joint" type="fixed">
     <parent link="chassis_link" />
-    <child link="navsat_link" />
+    <child link="gps" />
     <origin xyz="0 0 0" rpy="0 0 0" />
   </joint>

Commit message: fixed exports. updated with gps converter.

File: SC-LIO-SAM/launch/include/config/robot.urdf.xacro (robot description, xacro)
@@ -9,8 +9,8 @@
     <origin xyz="0 0 0" rpy="0 0 0" />
   </joint>
-  <link name="sensor"> </link>
+  <link name="imu_corrected"> </link>
   <joint name="imu_joint" type="fixed">
     <parent link="chassis_link" />
-    <child link="sensor" />
+    <child link="imu_corrected" />
     <origin xyz="0 0 0" rpy="0 0 0" />
   </joint>
